File: usb-c-expresscard.kicad_pcb (KiCad board)
At the start: 2 copper layers, 9.2 x 7 mm, 16 parts, among them J1 ExpressCard, J2 USB_C_Receptacle_USB2.0, U1 TPS61090, U2 TPS25821

Commit message: r1
Parts:
- added 3V3: TestPoint, TestPoint:TestPoint_Pad_D2.0mm, F.Cu at (149.3, 91.5)
- added 5V: TestPoint, TestPoint:TestPoint_Pad_D2.0mm, F.Cu at (178.0, 89.0)
- added GND: TestPoint, TestPoint:TestPoint_Pad_D2.0mm, F.Cu at (149.5, 84.5)
- added VBUS: TestPoint, TestPoint:TestPoint_Pad_D2.0mm, F.Cu at (185.0, 89.0)
- added kibuzzard-65DE897E: G***, kibuzzard-65DE897E, F.Cu at (181.2, 104.0)
- added kibuzzard-65DE8A1F: G***, kibuzzard-65DE8A1F, F.Cu at (149.8, 99.5)
- added kibuzzard-65DE8A3E: G***, kibuzzard-65DE8A3E, F.Cu at (151.1, 99.8)
- added kibuzzard-65DE8B98: G***, kibuzzard-65DE8B98, B.Cu at (171.3, 87.2)
- added kibuzzard-65DE8C34: G***, kibuzzard-65DE8C34, B.Cu at (162.8, 83.0)
- added kibuzzard-65DE8EC7: G***, kibuzzard-65DE8EC7, F.Cu at (146.4, 104.5)
- added kibuzzard-65DE8EF4: G***, kibuzzard-65DE8EF4, F.Cu at (150.3, 105.5)
- added kibuzzard-65DE8F1B: G***, kibuzzard-65DE8F1B, F.Cu at (156.9, 82.1)
- added kibuzzard-65DE8FDD: G***, kibuzzard-65DE8FDD, B.Cu at (177.1, 105.2)
- moved C5 75.2 mm to (173.8, 95.0), turned to 90 degrees
- moved R5 74.1 mm to (178.0, 99.3), turned to -90 degrees
- moved R6 72.9 mm to (181.0, 99.3), turned to -90 degrees
- moved C4 72.2 mm to (168.5, 95.0), turned to 90 degrees
- moved C3 66.8 mm to (168.2, 102.0), turned to -90 degrees
- moved J2 61.7 mm to (193.8, 94.5), turned to 90 degrees
- moved R3 59.5 mm to (164.5, 102.0), turned to -90 degrees
- moved R4 56.8 mm to (161.1, 102.0), turned to 90 degrees
- moved U2 53.0 mm to (180.5, 93.8)
- moved C1 48.7 mm to (154.5, 94.8), turned to -90 degrees
- moved C2 46.3 mm to (157.0, 94.8), turned to -90 degrees
- moved R2 45.0 mm to (147.1, 100.8), turned to 180 degrees
- moved U1 44.5 mm to (162.5, 97.0), turned to 180 degrees
- moved R1 41.5 mm to (147.1, 98.0), turned to 180 degrees
- moved J1 25.0 mm to (142.5, 106.5), turned to 180 degrees
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Connections:
- J2 pad S2: (no net) -> GND
- J2 pad S3: (no net) -> GND
- J2 pad S4: (no net) -> GND
Routing:
- net /D+: track 0.00 -> 60.6 mm, vias 0 -> 2
- net /D-: track 0.00 -> 59.6 mm, vias 0 -> 2
- net +3.3V: track 0.00 -> 34.9 mm
- net +5V: track 0.00 -> 34.6 mm
- net /VBUS: track 0.00 -> 32.0 mm, vias 0 -> 2
- net GND: track 0.00 -> 20.1 mm, vias 0 -> 21
- net Net-(J2-PadA5): track 0.00 -> 12.3 mm, vias 0 -> 2
- net Net-(J1-Pad12): track 0.00 -> 9.29 mm
- net Net-(L1-Pad1): track 0.00 -> 9.08 mm
- net Net-(R5-Pad2): track 0.00 -> 7.59 mm
- net Net-(J2-PadB5): track 0.00 -> 7.31 mm
- net Net-(R3-Pad2): track 0.00 -> 7.19 mm
- net Net-(R6-Pad1): track 0.00 -> 4.91 mm
- net Net-(J1-Pad8): track 0.00 -> 4.30 mm
- net Net-(J1-Pad7): track 0.00 -> 3.78 mm
- added copper zone on B.Cu, net GND
- added copper zone on F.Cu, net GND
Other:
- board size 9.2 x 7 mm -> 54.9 x 28 mm
- board text added: "L1: 6.8uH R1,R2: 5k C1: 10uF C2: 0.1uF R3: 1.87M R4: 200k C3: 2.2uF C4,C5: 100uF R5,R6: 100k"
- board text added: "TAHNOK"
- board text added: "WHAT? USB 2.0 from expresscard to USB-C connector Boost 3.3V to 5V Handle USB-C power shenanigans"
