File: usb-c-expresscard.kicad_sch (KiCad schematic)
At the start: 16 parts, among them J1 ExpressCard, J2 USB_C_Receptacle_USB2.0, U1 TPS61090, U2 TPS25821

Commit message: r1
Parts:
- added TP1, TP2, TP3, TP4: TestPoint, TestPoint:TestPoint_Pad_D2.0mm, symbol Connector:TestPoint
- C1, C2, C3: Digikey (none) -> https://www.digikey.ca/en/products/detail/samsung-electro-m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
- J2: Digikey (none) -> https://www.digikey.ca/en/products/detail/molex/2169900003/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
- R1, R2: Digikey (none) -> https://www.digikey.ca/en/products/detail/yageo/RT0603BRE07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
- R3: Digikey (none) -> https://www.digikey.ca/en/products/detail/stackpole-electro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
- R4, R5, R6: Digikey (none) -> https://www.digikey.ca/en/products/detail/yageo/RC0603FR-07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
- U1, U2: Digikey (none) -> https://www.digikey.ca/en/products/detail/texas-instruments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
Connections:
- net +3.3V: now also TP1.1
- net +5V: now also TP2.1
- net GND: now also TP4.1
- net VBUS: now also TP3.1
Other:
- title: (none) -> ExpressCard to USB-C
- moved on the sheet: C1, C2, C3, C4, C5, J1, J2, L1, R1, R2, R3, R4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
